Commit message: Add files via upload

File: urdf/hrp4.urdf (robot description, URDF)
Before this commit: robot hrp4, 66 links, 65 joints
Links:
- link CHEST_P_LINK: geometry collision mesh filename=../meshes/CHEST_P.dae; collision mesh filename=../meshes/CHEST_P.dae
- link L_ANKLE_P_LINK: geometry collision mesh filename=../meshes/L_ANKLE_P.dae; visual mesh filename=../meshes/L_ANKLE_P.dae
- link L_ANKLE_R_LINK: geometry collision mesh filename=../meshes/L_ANKLE_R.dae; visual mesh filename=../meshes/L_ANKLE_R.dae
- link L_ELBOW_P_LINK: geometry collision mesh filename=../meshes/ELBOW_P.dae; visual mesh filename=../meshes/ELBOW_P.dae
- link L_F22_LINK: geometry collision mesh filename=../meshes/F2.dae; visual mesh filename=../meshes/F2.dae
- link L_F23_LINK: geometry collision mesh filename=../meshes/F3.dae; visual mesh filename=../meshes/F3.dae
- link L_F32_LINK: geometry collision mesh filename=../meshes/F2.dae; visual mesh filename=../meshes/F2.dae
- link L_F33_LINK: geometry collision mesh filename=../meshes/F3.dae; visual mesh filename=../meshes/F3.dae
- link L_F42_LINK: geometry collision mesh filename=../meshes/F2.dae; visual mesh filename=../meshes/F2.dae
- link L_F43_LINK: geometry collision mesh filename=../meshes/F3.dae; visual mesh filename=../meshes/F3.dae
- link L_F52_LINK: geometry collision mesh filename=../meshes/F2.dae; visual mesh filename=../meshes/F2.dae
- link L_F53_LINK: geometry collision mesh filename=../meshes/F3.dae; visual mesh filename=../meshes/F3.dae
- link L_HAND_J0_LINK: geometry collision mesh filename=../meshes/L_THUMB.dae; visual mesh filename=../meshes/L_THUMB.dae
- link L_HAND_J1_LINK: geometry collision mesh filename=../meshes/L_F1.dae; visual mesh filename=../meshes/L_F1.dae
- link L_HIP_P_LINK: geometry collision mesh filename=../meshes/L_HIP_P.dae; visual mesh filename=../meshes/L_HIP_P.dae
- link L_HIP_R_LINK: geometry collision mesh filename=../meshes/CHEST_P.dae; visual mesh filename=../meshes/CHEST_P.dae
- link L_HIP_Y_LINK: geometry collision mesh filename=../meshes/HIP_Y.dae; visual mesh filename=../meshes/HIP_Y.dae
- link L_KNEE_P_LINK: geometry collision mesh filename=../meshes/L_KNEE_P.dae; visual mesh filename=../meshes/L_KNEE_P.dae
- link L_SHOULDER_P_LINK: geometry collision mesh filename=../meshes/L_SHOULDER_P.dae; visual mesh filename=../meshes/L_SHOULDER_P.dae
- link L_SHOULDER_R_LINK: geometry collision mesh filename=../meshes/L_SHOULDER_R.dae; visual mesh filename=../meshes/L_SHOULDER_R.dae
- link L_SHOULDER_Y_LINK: geometry collision mesh filename=../meshes/SHOULDER_Y.dae; visual mesh filename=../meshes/SHOULDER_Y.dae
- link L_WRIST_P_LINK: geometry collision mesh filename=../meshes/WRIST_P.dae; visual mesh filename=../meshes/WRIST_P.dae
- link L_WRIST_Y_LINK: geometry collision mesh filename=../meshes/L_WRIST_Y.dae; visual mesh filename=../meshes/L_WRIST_Y.dae
- link NECK_P_LINK: geometry collision mesh filename=../meshes/NECK_P.dae; visual mesh filename=../meshes/NECK_P.dae
- link NECK_Y_LINK: geometry collision mesh filename=../meshes/NECK_Y.dae; visual mesh filename=../meshes/NECK_Y.dae
- link R_ANKLE_P_LINK: geometry collision mesh filename=../meshes/L_ANKLE_P.dae; visual mesh filename=../meshes/L_ANKLE_P.dae
- link R_ANKLE_R_LINK: geometry collision mesh filename=../meshes/R_ANKLE_R.dae; visual mesh filename=../meshes/R_ANKLE_R.dae
- link R_ELBOW_P_LINK: geometry collision mesh filename=../meshes/ELBOW_P.dae; visual mesh filename=../meshes/ELBOW_P.dae
- link R_F22_LINK: geometry collision mesh filename=../meshes/F2.dae; visual mesh filename=../meshes/F2.dae
- link R_F23_LINK: geometry collision mesh filename=../meshes/F3.dae; visual mesh filename=../meshes/F3.dae
- link R_F32_LINK: geometry collision mesh filename=../meshes/F2.dae; visual mesh filename=../meshes/F2.dae
- link R_F33_LINK: geometry collision mesh filename=../meshes/F3.dae; visual mesh filename=../meshes/F3.dae
- link R_F42_LINK: geometry collision mesh filename=../meshes/F2.dae; visual mesh filename=../meshes/F2.dae
- link R_F43_LINK: geometry collision mesh filename=../meshes/F3.dae; visual mesh filename=../meshes/F3.dae
- link R_F52_LINK: geometry collision mesh filename=../meshes/F2.dae; visual mesh filename=../meshes/F2.dae
- link R_F53_LINK: geometry collision mesh filename=../meshes/F3.dae; visual mesh filename=../meshes/F3.dae
- link R_HAND_J0_LINK: geometry collision mesh filename=../meshes/R_THUMB.dae; visual mesh filename=../meshes/R_THUMB.dae
- link R_HAND_J1_LINK: geometry collision mesh filename=../meshes/R_F1.dae; visual mesh filename=../meshes/R_F1.dae
- link R_HIP_P_LINK: geometry collision mesh filename=../meshes/R_HIP_P.dae; visual mesh filename=../meshes/R_HIP_P.dae
- link R_HIP_R_LINK: geometry collision mesh filename=../meshes/CHEST_P.dae; visual mesh filename=../meshes/CHEST_P.dae
- link R_HIP_Y_LINK: geometry collision mesh filename=../meshes/HIP_Y.dae; visual mesh filename=../meshes/HIP_Y.dae
- link R_KNEE_P_LINK: geometry collision mesh filename=../meshes/R_KNEE_P.dae; visual mesh filename=../meshes/R_KNEE_P.dae
- link R_SHOULDER_P_LINK: geometry collision mesh filename=../meshes/R_SHOULDER_P.dae; visual mesh filename=../meshes/R_SHOULDER_P.dae
- link R_SHOULDER_R_LINK: geometry collision mesh filename=../meshes/R_SHOULDER_R.dae; visual mesh filename=../meshes/R_SHOULDER_R.dae
- link R_SHOULDER_Y_LINK: geometry collision mesh filename=../meshes/SHOULDER_Y.dae; visual mesh filename=../meshes/SHOULDER_Y.dae
- link R_WRIST_P_LINK: geometry collision mesh filename=../meshes/WRIST_P.dae; visual mesh filename=../meshes/WRIST_P.dae
- link R_WRIST_Y_LINK: geometry collision mesh filename=../meshes/R_WRIST_Y.dae; visual mesh filename=../meshes/R_WRIST_Y.dae
- link body: geometry collision mesh filename=../meshes/WAIST_LINK.dae; visual mesh filename=../meshes/WAIST_LINK.dae
- link l_ankle: geometry collision mesh filename=../meshes/L_FOOT.dae; visual mesh filename=../meshes/L_FOOT.dae
- link l_sole: mass None -> 2e-06; geometry collision box size=0.14 0.078 0.007; visual box size=0.14 0.078 0.007
- link l_wrist: geometry collision mesh filename=../meshes/L_WRIST_R.dae; visual mesh filename=../meshes/L_WRIST_R.dae
- link r_ankle: geometry collision mesh filename=../meshes/R_FOOT.dae; visual mesh filename=../meshes/R_FOOT.dae
- link r_sole: mass None -> 2e-06; geometry collision box size=0.14 0.078 0.007; visual box size=0.14 0.078 0.007
- link r_wrist: geometry collision mesh filename=../meshes/R_WRIST_R.dae; visual mesh filename=../meshes/R_WRIST_R.dae
- link torso: geometry collision mesh filename=../meshes/CHEST_Y.dae; visual mesh filename=../meshes/CHEST_Y.dae
